File: kicad/foxtemp2024-r1/foxtemp2024.kicad_pcb (KiCad board)
At the start: 2 copper layers, 33.5 x 70.8 mm, 29 parts, among them J1 AVR-ISP-6-PinHead, J2 Connector for Wire Antenna, J3 AVR-ISP-6-TagConn, J4 Conn_01x09, J5 Conn_01x07, U1 MAX17224ELT+T, U2 SHT4x, U4 ATmega328P-A, U5 RFM69HCW

Commit message: revision 1 as sent to JLCPCB for production
Parts:
- added C99: optional1, Capacitor_THT:CP_Radial_D6.3mm_P2.50mm, F.Cu at (108.3, 86.6)
Routing:
- net GND: track 78.6 -> 81.6 mm, vias 28 -> 29
- net +3V3: track 170.2 -> 171.2 mm
