File: kicad/foxtemp2024-r1/foxtemp2024.kicad_sch (KiCad schematic)
At the start: 29 parts, among them J1 AVR-ISP-6-PinHead, J2 Connector for Wire Antenna, J3 AVR-ISP-6-TagConn, J4 Conn_01x09, J5 Conn_01x07, U1 MAX17224ELT+T, U2 SHT4x, U4 ATmega328P-A, U5 RFM69HCW

Commit message: revision 1 as sent to JLCPCB for production
Parts:
- added C99: optional1, Capacitor_THT:CP_Radial_D6.3mm_P2.50mm, symbol Device:C_Polarized
Connections:
- net +3V3: now also C99.1
- net GND: now also C99.2
Other:
- moved on the sheet: BAT1
